File: eagle/tfpcmcia.sch (EAGLE design)
At the start: 44 parts, among them IC1 CH32V307, IC2 LM1117MPX-3.3, IC3 APS6404L, IC4 MCP6001RT-I_OT, J2 MSD-11-A

Commit message: Board updates for revision 1
Parts:
- added JP1, JP2: (no value), SparkFun-Retired:JUMPER-2PTH
- added R7: 2K2, rcl:R-EU_R0603
- R1: value 10k -> 2K2
Connections:
- new net BOOT0: IC1.BOOT0, JP2.1, R7.2
- new net USB1_DM: IC1.PA11, JP1.2
- new net USB1_DP: IC1.PA12, JP1.1
- net GND: now also R7.1; no longer IC1.BOOT0
- net RAM_MISO: now also IC1.PA6; no longer IC1.PA7
- net RAM_MOSI: now also IC1.PA7; no longer IC1.PA6
- net VCC33: now also JP2.2
Changed lines of the file:
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@@
 <part name="C3" library="rcl" library_urn="urn:adsk.eagle:library:334" deviceset="C-EU" device="C1206" package3d_urn="urn:adsk.eagle:package:23618/2" value="1uF"/>
 <part name="PWR" library="led" library_urn="urn:adsk.eagle:library:259" deviceset="LED" device="SML0805" package3d_urn="urn:adsk.eagle:package:15830/1" value="LED"/>
-<part name="R1" library="rcl" library_urn="urn:adsk.eagle:library:334" deviceset="R-EU_" device="R0603" package3d_urn="urn:adsk.eagle:package:23555/3" value="10k"/>
+<part name="R1" library="rcl" library_urn="urn:adsk.eagle:library:334" deviceset="R-EU_" device="R0603" package3d_urn="urn:adsk.eagle:package:23555/3" value="2K2"/>
 <part name="DEBUG" library="microbuilder" deviceset="HEADER-1X6" device="ROUND" value="JTAG"/>
 <part name="J2" library="SamacSys_Parts" deviceset="MSD-11-A" device=""/>
@@
 <part name="LED8" library="Blinkenlights" deviceset="COM-14608" device=""/>
 <part name="LED9" library="Blinkenlights" deviceset="COM-14608" device=""/>
+<part name="JP1" library="SparkFun-Retired" library_urn="urn:adsk.eagle:library:533" deviceset="JUMPER-2" device="PTH" package3d_urn="urn:adsk.eagle:package:41385954/1"/>
+<part name="JP2" library="SparkFun-Retired" library_urn="urn:adsk.eagle:library:533" deviceset="JUMPER-2" device="PTH" package3d_urn="urn:adsk.eagle:package:41385954/1"/>
+<part name="R7" library="rcl" library_urn="urn:adsk.eagle:library:334" deviceset="R-EU_" device="R0603" package3d_urn="urn:adsk.eagle:package:23555/3" value="2K2"/>
 </parts>
 <sheets>
@@
 <attribute name="VALUE" x="273.05" y="177.8" size="1.778" layer="96" align="center-left"/>
 </instance>
+<instance part="JP1" gate="A" x="223.52" y="73.66" smashed="yes" rot="R270">
+<attribute name="NAME" x="223.52" y="74.93" size="1.778" layer="95"/>
+<attribute name="VALUE" x="223.52" y="67.945" size="1.778" layer="96"/>
+</instance>
+<instance part="JP2" gate="A" x="83.82" y="116.84" smashed="yes" rot="R180">
+<attribute name="NAME" x="85.09" y="116.84" size="1.778" layer="95" rot="R270"/>
+<attribute name="VALUE" x="78.105" y="116.84" size="1.778" layer="96" rot="R270"/>
+</instance>
+<instance part="R7" gate="G$1" x="91.44" y="132.08" smashed="yes" rot="R270">
+<attribute name="NAME" x="92.9386" y="135.89" size="1.778" layer="95" rot="R270"/>
+<attribute name="VALUE" x="88.138" y="135.89" size="1.778" layer="96" rot="R270"/>
+</instance>
 </instances>
 <busses>
@@
 </segment>
 </bus>
-<bus name="A[0..31],AUD_MIXED,AUD_O,BVD[1..2],CD[1..2],CE[1..2],D[0..15],GND,IORD,IOWR,LED[1..3],LED_CLK,LED_DO,NRST,OE,RAM_CLK,RAM_MISO,RAM_MOSI,RAM_SNSS,READY,!REG,RESET,SD_CD,SD_CLK,SD_MISO,SD_MOSI,SD_SNSS,SWCLK,SWDIO,USART_RX,USART_TX,VCC,VCC33,!VS[1..2],!WAIT,!WE,WP/!IOCS16">
+<bus name="A[0..31],AUD_MIXED,AUD_O,BOOT0,BVD[1..2],CD[1..2],CE[1..2],D[0..15],GND,IORD,IOWR,LED[1..3],LED_CLK,LED_DO,NRST,OE,RAM_CLK,RAM_MISO,RAM_MOSI,RAM_SNSS,READY,!REG,RESET,SD_CD,SD_CLK,SD_MISO,SD_MOSI,SD_SNSS,SWCLK,SWDIO,USART_RX,USART_TX,USB1_DM,USB1_DP,VCC,VCC33,!VS[1..2],!WAIT,!WE,WP/!IOCS16">
 <segment>
 <wire x1="63.5" y1="142.24" x2="63.5" y2="-2.54" width="0.762" layer="92"/>
@@
 </segment>
 <segment>
-<pinref part="IC1" gate="G$1" pin="BOOT0"/>
-<wire x1="119.38" y1="119.38" x2="119.38" y2="142.24" width="0.1524" layer="91"/>
-<label x="119.38" y="124.46" size="1.778" layer="95" rot="R90"/>
-</segment>
-<segment>
 <pinref part="LED3" gate="G$1" pin="GND"/>
 <wire x1="17.78" y1="167.64" x2="10.16" y2="167.64" width="0.1524" layer="91"/>
@@
 <wire x1="248.92" y1="167.64" x2="246.38" y2="167.64" width="0.1524" layer="91"/>
 <wire x1="246.38" y1="167.64" x2="246.38" y2="157.48" width="0.1524" layer="91"/>
+</segment>
+<segment>
+<pinref part="R7" gate="G$1" pin="1"/>
+<wire x1="91.44" y1="137.16" x2="91.44" y2="142.24" width="0.1524" layer="91"/>
 </segment>
 </net>
@@
 <label x="340.36" y="142.24" size="1.778" layer="95"/>
 </segment>
+<segment>
+<pinref part="JP2" gate="A" pin="2"/>
+<wire x1="81.28" y1="119.38" x2="81.28" y2="142.24" width="0.1524" layer="91"/>
+<label x="81.28" y="129.54" size="1.778" layer="95" rot="R90"/>
+</segment>
 </net>
 <net name="USART_RX" class="0">
@@
 <net name="RAM_MOSI" class="0">
 <segment>
-<pinref part="IC1" gate="G$1" pin="PA6"/>
-<wire x1="116.84" y1="22.86" x2="116.84" y2="-2.54" width="0.1524" layer="91"/>
-<label x="116.84" y="2.54" size="1.778" layer="95" rot="R90"/>
-</segment>
-<segment>
 <pinref part="IC3" gate="G$1" pin="MOSI"/>
 <wire x1="294.64" y1="33.02" x2="297.18" y2="33.02" width="0.1524" layer="91"/>
 <label x="297.18" y="33.02" size="1.27" layer="95" xref="yes"/>
 </segment>
+<segment>
+<wire x1="119.38" y1="22.86" x2="119.38" y2="-2.54" width="0.1524" layer="91"/>
+<pinref part="IC1" gate="G$1" pin="PA7"/>
+<label x="119.38" y="2.54" size="1.778" layer="95" rot="R90"/>
+</segment>
 </net>
 <net name="RAM_MISO" class="0">
-<segment>
-<pinref part="IC1" gate="G$1" pin="PA7"/>
-<wire x1="119.38" y1="22.86" x2="119.38" y2="-2.54" width="0.1524" layer="91"/>
-<label x="119.38" y="2.54" size="1.778" layer="95" rot="R90"/>
-</segment>
 <segment>
 <pinref part="IC3" gate="G$1" pin="MISO"/>
 <wire x1="264.16" y1="38.1" x2="261.62" y2="38.1" width="0.1524" layer="91"/>
 <label x="261.62" y="38.1" size="1.27" layer="95" rot="R180" xref="yes"/>
+</segment>
+<segment>
+<wire x1="116.84" y1="22.86" x2="116.84" y2="-2.54" width="0.1524" layer="91"/>
+<pinref part="IC1" gate="G$1" pin="PA6"/>
+<label x="116.84" y="2.54" size="1.778" layer="95" rot="R90"/>
 </segment>
 </net>
@@
 </segment>
 </net>
+<net name="USB1_DP" class="0">
+<segment>
+<pinref part="IC1" gate="G$1" pin="PA12"/>
+<wire x1="172.72" y1="91.44" x2="205.74" y2="91.44" width="0.1524" layer="91"/>
+<label x="187.96" y="91.44" size="1.778" layer="95"/>
+</segment>
+<segment>
+<pinref part="JP1" gate="A" pin="1"/>
+<wire x1="220.98" y1="73.66" x2="205.74" y2="73.66" width="0.1524" layer="91"/>
+<label x="208.28" y="73.66" size="1.778" layer="95"/>
+</segment>
+</net>
+<net name="USB1_DM" class="0">
+<segment>
+<pinref part="IC1" gate="G$1" pin="PA11"/>
+<wire x1="172.72" y1="88.9" x2="205.74" y2="88.9" width="0.1524" layer="91"/>
+<label x="187.96" y="88.9" size="1.778" layer="95"/>
+</segment>
+<segment>
+<pinref part="JP1" gate="A" pin="2"/>
+<wire x1="220.98" y1="71.12" x2="205.74" y2="71.12" width="0.1524" layer="91"/>
+<label x="208.28" y="71.12" size="1.778" layer="95"/>
+</segment>
+</net>
+<net name="BOOT0" class="0">
+<segment>
+<pinref part="IC1" gate="G$1" pin="BOOT0"/>
+<wire x1="119.38" y1="119.38" x2="119.38" y2="142.24" width="0.1524" layer="91"/>
+<label x="119.38" y="124.46" size="1.778" layer="95" rot="R90"/>
+</segment>
+<segment>
+<pinref part="JP2" gate="A" pin="1"/>
+<label x="83.82" y="129.54" size="1.778" layer="95" rot="R90"/>
+<wire x1="83.82" y1="119.38" x2="83.82" y2="121.92" width="0.1524" layer="91"/>
+<pinref part="R7" gate="G$1" pin="2"/>
+<wire x1="83.82" y1="121.92" x2="83.82" y2="142.24" width="0.1524" layer="91"/>
+<wire x1="91.44" y1="127" x2="91.44" y2="121.92" width="0.1524" layer="91"/>
+<wire x1="91.44" y1="121.92" x2="83.82" y2="121.92" width="0.1524" layer="91"/>
+<junction x="83.82" y="121.92"/>
+</segment>
+</net>
