File: eagle/tfpcmcia.sch (EAGLE design)
At the start: 47 parts, among them IC1 CH32V307, IC2 LM1117MPX-3.3, IC3 APS6404L, IC4 MCP6001RT-I_OT, J2 MSD-11-A

Commit message: CH32V467 upgrade
Parts:
- removed C17, C19: 1uF, eagle-ltspice:CC0603
- removed C18: 100nF, eagle-ltspice:CC0603
- removed IC3: APS6404L, SparkFun-IC-Memory:SPI_FLASH-X25XXSMD
- removed IC4: MCP6001RT-I_OT, SamacSys_Parts:MCP6001RT-I_OT
- removed JP1: (no value), SparkFun-Retired:JUMPER-2PTH
- removed R4, R5, R6: 10k, rcl:R-EU_R0603
- added LED10: COM-14608, Blinkenlights:COM-14608
- C13: value 4.7uF -> 100nF
- C14: value 4.7uF -> 2.2uF
- C15: value 1nF -> 2.2uF
- C16: value 1nF -> 22uF; device eagle-ltspice:CC0603 -> rcl:C-EUC1206
- IC1: value CH32V307 -> CH32V467; device SamacSys_Parts:STM32F103VET6 -> SamacSys_Parts:CH32V467VET6
Connections:
- removed net AUD_MIXED: C14.1, IC1.PA4
- removed net AUD_O: C13.1, PCMCIA.62
- removed net N$10: C15.1, IC4.VIN-, R4.2, R6.1
- removed net N$7: C13.2, C15.2, IC4.VOUT, R6.2
- removed net N$8: C16.1, IC4.VIN+, R5.1
- removed net N$9: C14.2, R5.2
- removed net RAM_CLK: IC1.PA5, IC3.SCK
- removed net RAM_MISO: IC1.PA6, IC3.MISO
- removed net RAM_MOSI: IC1.PA7, IC3.MOSI
- removed net RAM_SNSS: IC1.PA1, IC3.CS
- removed net USB1_DM: IC1.PA11, JP1.2
- removed net USB1_DP: IC1.PA12, JP1.1
- new net VDD18: C13.1, C14.1, IC1.VDD18
- new net VDDK: C15.1, C4.1, IC1.VDDK
- net !REG: now also IC1.PC10; no longer IC1.PB10
- net !WAIT: now also IC1.PA8; no longer IC1.PB14
- net !WE: now also IC1.PC8; no longer IC1.PB8
- net A12: now also IC1.PB8; no longer IC1.PE12
- net A13: now also IC1.PB9; no longer IC1.PE13
- net A14: now also IC1.PB10; no longer IC1.PE14
- net A15: now also IC1.PB11; no longer IC1.PE15
- net A16: now also IC1.PB12; no longer IC1.PB0
- net A17: now also IC1.PB13; no longer IC1.PB1
- net A18: now also IC1.PB14; no longer IC1.PB2
- net A19: now also IC1.PB15; no longer IC1.PB3
- net A7: now also IC1.PB3; no longer IC1.PE7
- net BOOT0: now also IC1.PE12-BOOT0; no longer IC1.BOOT0
- net CE1: now also IC1.PC6; no longer IC1.PB6
- net CE2: now also IC1.PC9; no longer IC1.PB9
- net GND: now also C13.2, C14.2, C15.2, IC1.VSS_4, LED10.GND; no longer C17.2, C18.2, C19.2, IC3.GND, IC4.VSS, R4.1
- net IORD: now also IC1.PC11; no longer IC1.PB11
- net IOWR: now also IC1.PC12; no longer IC1.PB12
- net LED1: now also IC1.PB0; no longer IC1.PC8
- net LED2: now also IC1.PB1; no longer IC1.PC7
- net N$3: now also LED10.CIN, LED9.COUT; no longer IC3.HOLD, RN1.2
- net N$4: now also LED10.DIN, LED9.DOUT; no longer IC3.WP, RN1.1
- net OE: now also IC1.PC7; no longer IC1.PB7
- net READY: now also IC1.PA9; no longer IC1.PA2
- net RESET: now also IC1.PA15; no longer IC1.PB13
- net SD_CD: now also IC1.PC5; no longer IC1.PA15
- net SD_CLK: now also IC1.PA5; no longer IC1.PC10
- net SD_MISO: now also IC1.PA6; no longer IC1.PC11
- net SD_MOSI: now also IC1.PA7; no longer IC1.PC12
- net SD_SNSS: now also IC1.PC4; no longer IC1.PC9
- net USART_RX: now also IC1.PB7; no longer IC1.PA10
- net USART_TX: now also IC1.PB6; no longer IC1.PA9
- net VCC: now also LED10.VCC; no longer C17.1, C18.1, IC4.VDD
- net VCC33: now also C16.1, IC1.VDD_4, IC1.VDD_MAIN; no longer C19.1, C4.1, IC1.VDD_5, IC3.VCC
- net WP/!IOCS16: now also IC1.PA10; no longer IC1.PB15
Other:
- note removed: "IC3 is SPI RAM."
- note removed: "Unfortunately the CH32 chips dont do QUAD SPI."
- moved on the sheet: C13, C14, C15, C16, C4
