File: eagle/tfpcmcia.sch (EAGLE design)
At the start: 39 parts, among them IC1 CH32V467, IC2 LM1117MPX-3.3, J2 MSD-11-A

Commit message: CH32V467 upgrade
Parts:
- added C17, C18: 100nF, eagle-ltspice:CC0603
Connections:
- net GND: now also C17.2, C18.2
- net VCC33: now also C17.1, C18.1
Changed lines of the file:
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@@
 <part name="C15" library="eagle-ltspice" deviceset="C" device="C0603" value="2.2uF"/>
 <part name="C16" library="rcl" library_urn="urn:adsk.eagle:library:334" deviceset="C-EU" device="C1206" package3d_urn="urn:adsk.eagle:package:23618/2" value="22uF"/>
+<part name="C17" library="eagle-ltspice" deviceset="C" device="C0603" value="100nF"/>
+<part name="C18" library="eagle-ltspice" deviceset="C" device="C0603" value="100nF"/>
 </parts>
 <sheets>
@@
 <attribute name="NAME" x="301.244" y="96.901" size="1.778" layer="95"/>
 <attribute name="VALUE" x="301.244" y="91.821" size="1.778" layer="96"/>
+</instance>
+<instance part="C17" gate="G$1" x="307.34" y="142.24" smashed="yes">
+<attribute name="NAME" x="308.864" y="142.621" size="1.778" layer="95"/>
+<attribute name="VALUE" x="308.864" y="137.541" size="1.778" layer="96"/>
+</instance>
+<instance part="C18" gate="G$1" x="236.22" y="142.24" smashed="yes">
+<attribute name="NAME" x="237.744" y="142.621" size="1.778" layer="95"/>
+<attribute name="VALUE" x="237.744" y="137.541" size="1.778" layer="96"/>
 </instance>
 </instances>
@@
 <wire x1="307.34" y1="127" x2="307.34" y2="137.16" width="0.1524" layer="91"/>
 <junction x="297.18" y="127"/>
+<pinref part="C17" gate="G$1" pin="2"/>
+<pinref part="C18" gate="G$1" pin="2"/>
+<wire x1="236.22" y1="137.16" x2="236.22" y2="127" width="0.1524" layer="91"/>
 </segment>
 <segment>
@@
 <wire x1="307.34" y1="152.4" x2="307.34" y2="144.78" width="0.1524" layer="91"/>
 <junction x="297.18" y="152.4"/>
-</segment>
-<segment>
+<pinref part="C17" gate="G$1" pin="1"/>
+<pinref part="C18" gate="G$1" pin="1"/>
+<wire x1="236.22" y1="152.4" x2="236.22" y2="144.78" width="0.1524" layer="91"/>
+</segment>
+<segment>

Commit message: final updates
Parts:
- C1: value 100nF -> 1uF
- C3: value 1uF -> 10uF
Connections:
- net GND: now also IC1.PB2-BOOT1
Changed lines of the file:
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@@
 <part name="SUPPLY2" library="supply2" library_urn="urn:adsk.eagle:library:372" deviceset="VCC" device=""/>
 <part name="C2" library="eagle-ltspice" deviceset="C" device="C0603" value="10uF"/>
-<part name="C1" library="rcl" library_urn="urn:adsk.eagle:library:334" deviceset="C-EU" device="C1206" package3d_urn="urn:adsk.eagle:package:23618/2" value="100nF"/>
-<part name="C3" library="rcl" library_urn="urn:adsk.eagle:library:334" deviceset="C-EU" device="C1206" package3d_urn="urn:adsk.eagle:package:23618/2" value="1uF"/>
+<part name="C1" library="rcl" library_urn="urn:adsk.eagle:library:334" deviceset="C-EU" device="C1206" package3d_urn="urn:adsk.eagle:package:23618/2" value="1uF"/>
+<part name="C3" library="rcl" library_urn="urn:adsk.eagle:library:334" deviceset="C-EU" device="C1206" package3d_urn="urn:adsk.eagle:package:23618/2" value="10uF"/>
 <part name="PWR" library="led" library_urn="urn:adsk.eagle:library:259" deviceset="LED" device="SML0805" package3d_urn="urn:adsk.eagle:package:15830/1" value="LED"/>
 <part name="R1" library="rcl" library_urn="urn:adsk.eagle:library:334" deviceset="R-EU_" device="R0603" package3d_urn="urn:adsk.eagle:package:23555/3" value="2K2"/>
@@
 <pinref part="C14" gate="G$1" pin="2"/>
 </segment>
+<segment>
+<pinref part="IC1" gate="G$1" pin="PB2-BOOT1"/>
+<wire x1="132.08" y1="22.86" x2="132.08" y2="-2.54" width="0.1524" layer="91"/>
+<label x="132.08" y="10.16" size="1.778" layer="95" rot="R90"/>
+</segment>
 </net>
