File: eagle/tfpcmcia.brd (EAGLE design)
At the start: 80.4 x 44.4 mm, 47 parts, among them IC1 CH32V307, IC2 LM1117MPX-3.3, IC3 APS6404L, IC4 MCP6001RT-I_OT, J2 MSD-11-A

Commit message: Board updates for revision 1
Routing:
- net GND: track 62.7 -> 63.3 mm
Changed lines of the file:
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@@
 <via x="77.0624375" y="22.353946875" extent="1-16" drill="0.35"/>
 <contactref element="R7" pad="1"/>
-<wire x1="48.50365625" y1="19.92145" x2="49.3441125" y2="19.92145" width="0.1524" layer="1"/>
-<wire x1="49.3441125" y1="19.92145" x2="49.35255625" y2="19.92989375" width="0.1524" layer="1"/>
-<via x="49.35255625" y="19.92989375" extent="1-16" drill="0.35"/>
+<wire x1="48.50365625" y1="19.92145" x2="48.50365625" y2="20.188590625" width="0.1524" layer="1"/>
+<wire x1="49.307484375" y1="20.99241875" x2="48.50365625" y2="20.188590625" width="0.1524" layer="1"/>
+<via x="49.307484375" y="20.99241875" extent="1-16" drill="0.35"/>
 </signal>
 <signal name="D3">
